File: Alpenglow_ChillySnowCloud_OnlySilverSnowflakes_PCB.kicad_pcb (KiCad board)
At the start: 2 copper layers, 52.4 x 52.4 mm, 10 parts, among them SW1 SW_SPDT

Commit message: Update Final Design
Other:
- net class Default removed
